File: projects/pzko_led/led_board.brd (EAGLE design)
At the start: 100 x 100 mm, 76 parts

Commit message: bee counter board
Parts:
- moved T3 1.00 mm to (35.0, 68.0)
Routing:
- net N$4: track 231.5 -> 232.5 mm
Changed lines of the file:
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@@
 <attribute name="VALUE" x="32.46" y="48.6792" size="1.27" layer="27"/>
 </element>
-<element name="T3" library="transistor-neu-to92" library_urn="urn:adsk.eagle:library:397" package="SOT223" package3d_urn="urn:adsk.eagle:package:28541/2" value="" x="34" y="68" smashed="yes">
-<attribute name="NAME" x="31.46" y="68.0508" size="1.27" layer="25"/>
-<attribute name="POPULARITY" value="0" x="34" y="68" size="1.778" layer="27" display="off"/>
-<attribute name="VALUE" x="31.46" y="66.6792" size="1.27" layer="27"/>
+<element name="T3" library="transistor-neu-to92" library_urn="urn:adsk.eagle:library:397" package="SOT223" package3d_urn="urn:adsk.eagle:package:28541/2" value="" x="35" y="68" smashed="yes">
+<attribute name="NAME" x="32.46" y="68.0508" size="1.27" layer="25"/>
+<attribute name="POPULARITY" value="0" x="35" y="68" size="1.778" layer="27" display="off"/>
+<attribute name="VALUE" x="32.46" y="66.6792" size="1.27" layer="27"/>
 </element>
 <element name="R5" library="rcl" library_urn="urn:adsk.eagle:library:334" package="M1206" package3d_urn="urn:adsk.eagle:package:23566/2" value="3k3" x="28" y="35" smashed="yes" rot="R270">
@@
 <wire x1="29.387421875" y1="62.6" x2="29.893709375" y2="63.106290625" width="1" layer="1"/>
 <contactref element="R32" pad="2"/>
-<wire x1="29.893709375" y1="63.106290625" x2="31.6886" y2="64.9012" width="1" layer="1"/>
-<wire x1="31.6" y1="62" x2="30.493709375" y2="63.106290625" width="1" layer="1"/>
+<wire x1="31.19370625" y1="63.40629375" x2="32.6886" y2="64.9012" width="1" layer="1"/>
+<wire x1="31.6" y1="62" x2="31.6" y2="63" width="1" layer="1"/>
+<wire x1="31.6" y1="63" x2="31.19370625" y2="63.40629375" width="1" layer="1"/>
 <wire x1="30.493709375" y1="63.106290625" x2="29.893709375" y2="63.106290625" width="1" layer="1"/>
 </signal>
@@
 <via x="76" y="29" extent="1-16" drill="1.2"/>
 <wire x1="76" y1="29" x2="61" y2="29" width="1" layer="16"/>
-<wire x1="34" y1="71.099" x2="33" y2="72.099" width="1" layer="1"/>
-<wire x1="33" y1="72.099" x2="7.901" y2="72.099" width="1" layer="1"/>
+<wire x1="35" y1="71.099" x2="34" y2="72.099" width="1" layer="1"/>
+<wire x1="34" y1="72.099" x2="7.901" y2="72.099" width="1" layer="1"/>
 <wire x1="7.901" y1="72.099" x2="6" y2="74" width="1" layer="1"/>
 <wire x1="6" y1="74" x2="6" y2="82" width="1" layer="1"/>
@@
 <wire x1="54" y1="35" x2="54" y2="33.5898" width="2" layer="1"/>
 <wire x1="54" y1="33.5898" x2="52.3114" y2="31.9012" width="2" layer="1"/>
-<wire x1="36.3114" y1="64.9012" x2="37.2126" y2="64" width="2" layer="1"/>
-<wire x1="37.2126" y1="64" x2="37.2126" y2="62" width="2" layer="1"/>
+<wire x1="37.3114" y1="64.9012" x2="37.2126" y2="64.8024" width="2" layer="1"/>
+<wire x1="37.2126" y1="64.8024" x2="37.2126" y2="62" width="2" layer="1"/>
 <wire x1="37.2126" y1="62" x2="37.2126" y2="59" width="2" layer="1"/>
 <wire x1="39" y1="53" x2="42" y2="53" width="2" layer="1"/>
