File: projects/tank_waldek_2_0/chassis_board.brd (EAGLE design)
At the start: 100 x 61 mm, 20 parts, among them U1 NUCLEO-L432KC

Commit message: added gnss, imu and barometer modules
Routing:
- net N$1: track 116.6 -> 123.9 mm
Changed lines of the file:
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@@
 <wire x1="17.51" y1="51.01" x2="26.72" y2="51.01" width="1" layer="1"/>
 <wire x1="26.72" y1="51.01" x2="28.48" y2="49.25" width="1" layer="1"/>
-<wire x1="35.29" y1="48.81" x2="38.71" y2="44.09" width="0" layer="19" extent="1-1"/>
+<wire x1="35.29" y1="48.81" x2="35.29" y2="46.71" width="1" layer="1"/>
+<wire x1="35.29" y1="46.71" x2="36" y2="46" width="1" layer="1"/>
+<wire x1="36" y1="46" x2="38" y2="46" width="1" layer="1"/>
+<wire x1="38" y1="46" x2="38.71" y2="45.29" width="1" layer="1"/>
+<wire x1="38.71" y1="45.29" x2="38.71" y2="44.09" width="1" layer="1"/>
 </signal>
 <signal name="N$2">

Commit message: fixed waldek missing pwm outputs, wop on gramofon
Parts:
- added X4, X5: (no value), con-wago-500:W237-102
- moved R2 17.5 mm to (55.3, 56.3), turned to 180 degrees
- moved LED2 14.4 mm to (61.7, 56.0), turned to 0 degrees
- moved JP4 10.0 mm to (89.5, 28.0)
- moved X3 9.00 mm to (76.0, 54.0)
- moved JP2 6.08 mm to (89.8, 17.0)
- moved X1 1.00 mm to (76.2, 4.65)
- moved X2 1.00 mm to (86.4, 4.65)
Connections:
- net GND: now also R1.1
- net N$1: no longer R1.1
- net PWM_LEFT_B: now also X5.1
- net PWM_LEFT_F: now also X5.2
- net PWM_RIGHT_B: now also X4.1
- net PWM_RIGHT_F: now also X4.2
Routing:
- net PWM_RIGHT_B: track 0.00 -> 66.8 mm, vias 0 -> 2
- net PWM_RIGHT_F: track 0.00 -> 64.9 mm, vias 0 -> 2
- net PWM_LEFT_B: track 0.00 -> 51.7 mm
- net PWM_LEFT_F: track 0.00 -> 50.0 mm
- net GND: track 254.5 -> 274.9 mm
- net VCC: track 132.6 -> 141.6 mm
- net SDA: track 35.6 -> 40.7 mm
- net SCL: track 36.1 -> 40.7 mm
- net SSEL: track 45.4 -> 48.9 mm
- net SCLK: track 19.6 -> 23.1 mm
- net MOSI: track 19.6 -> 23.1 mm
- net MISO: track 19.6 -> 23.1 mm
- net N$1: track 123.9 -> 127.1 mm, vias 0 -> 2
- net GPIO2: track 23.9 -> 23.2 mm
Other:
- board size 100 x 61 mm -> 100 x 60 mm
