File: projects/gramofon/main_board.brd (EAGLE design)
At the start: 290 x 99 mm, 2 parts

Commit message: fixed waldek missing pwm outputs, wop on gramofon
Parts:
- removed U$1: RIAA_PREAMP, ligocki:RIAA_PREAMP
- added U$2, U$3, U$4: BUTTON, gramofon:BUTTON
- added U$5: MOTOR_DRIVER, gramofon:MOTOR_DRIVER
Other:
- outline, holes or cut-outs redrawn
Changed lines of the file:
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@@
 <?xml version="1.0" encoding="utf-8"?>
 <!DOCTYPE eagle SYSTEM "eagle.dtd">
-<eagle version="9.3.2">
+<eagle version="9.6.2">
 <drawing>
 <settings>
@@
 <setting verticaltext="up"/>
 </settings>
-<grid distance="1" unitdist="mm" unit="mm" style="lines" multiple="1" display="no" altdistance="5" altunitdist="mil" altunit="mil"/>
+<grid distance="1" unitdist="mm" unit="mm" style="dots" multiple="1" display="yes" altdistance="5" altunitdist="mil" altunit="mil"/>
 <layers>
 <layer number="1" name="Top" color="4" fill="1" visible="yes" active="yes"/>
@@
 <wire x1="188" y1="87" x2="188" y2="99" width="0.1524" layer="20"/>
 <wire x1="188" y1="99" x2="290" y2="99" width="0.1524" layer="20"/>
-<wire x1="245" y1="84" x2="245" y2="34" width="0.1524" layer="20"/>
-<wire x1="245" y1="34" x2="232" y2="34" width="0.1524" layer="20"/>
-<wire x1="232" y1="34" x2="232" y2="84" width="0.1524" layer="20"/>
-<wire x1="232" y1="84" x2="245" y2="84" width="0.1524" layer="20"/>
+<wire x1="235" y1="84" x2="235" y2="34" width="0.1524" layer="20"/>
+<wire x1="235" y1="34" x2="222" y2="34" width="0.1524" layer="20"/>
+<wire x1="222" y1="34" x2="222" y2="84" width="0.1524" layer="20"/>
+<wire x1="222" y1="84" x2="235" y2="84" width="0.1524" layer="20"/>
 <hole x="263" y="94" drill="5"/>
 <hole x="263" y="6" drill="5"/>
@@
 <dimension x1="57" y1="86" x2="57" y2="99" x3="52" y3="92.5" textsize="1.778" layer="47"/>
 <dimension x1="162" y1="87" x2="188" y2="87" x3="175" y3="81" textsize="1.778" layer="47"/>
-<dimension x1="232" y1="34" x2="232" y2="84" x3="250" y3="59" textsize="1.778" layer="47"/>
-<dimension x1="232" y1="84" x2="245" y2="84" x3="238.5" y3="87" textsize="1.778" layer="47"/>
+<dimension x1="222" y1="34" x2="222" y2="84" x3="240" y3="59" textsize="1.778" layer="47"/>
+<dimension x1="222" y1="84" x2="235" y2="84" x3="228.5" y3="87" textsize="1.778" layer="47"/>
 <hole x="67" y="92" drill="5"/>
 <dimension x1="67" y1="92" x2="57" y2="92" x3="62" y3="86" textsize="1.778" layer="47"/>
@@
 <dimension x1="68" y1="5" x2="68" y2="0" x3="74" y3="2.5" textsize="1.778" layer="47"/>
 <dimension x1="188" y1="87" x2="188" y2="99" x3="194" y3="93" textsize="1.778" layer="47"/>
-<wire x1="232" y1="59" x2="232" y2="34" width="0.1524" layer="47"/>
-<dimension x1="232" y1="59" x2="232" y2="34" x3="238" y3="46.5" textsize="1.778" layer="47"/>
-<wire x1="232" y1="59" x2="217" y2="59" width="0.1524" layer="47"/>
-<dimension x1="232" y1="59" x2="217" y2="59" x3="224.5" y3="62" textsize="1.778" layer="47"/>
-<dimension x1="217" y1="69" x2="217" y2="59" x3="212" y3="64" textsize="1.778" layer="47" dtype="horizontal"/>
-<dimension x1="217" y1="49" x2="217" y2="59" x3="212" y3="54" textsize="1.778" layer="47" dtype="horizontal"/>
+<wire x1="222" y1="59" x2="222" y2="34" width="0.1524" layer="47"/>
+<dimension x1="222" y1="59" x2="222" y2="34" x3="228" y3="46.5" textsize="1.778" layer="47"/>
+<wire x1="222" y1="59" x2="207" y2="59" width="0.1524" layer="47"/>
+<dimension x1="222" y1="59" x2="207" y2="59" x3="214.5" y3="62" textsize="1.778" layer="47"/>
+<dimension x1="207" y1="69" x2="207" y2="59" x3="202" y3="64" textsize="1.778" layer="47" dtype="horizontal"/>
+<dimension x1="207" y1="49" x2="207" y2="59" x3="202" y3="54" textsize="1.778" layer="47" dtype="horizontal"/>
+<dimension x1="235" y1="34" x2="290" y2="34" x3="262.5" y3="30" textsize="1.778" layer="47"/>
+<dimension x1="235" y1="84" x2="245" y2="99" x3="246" y3="91.5" textsize="1.778" layer="47" dtype="vertical"/>
 </plain>
 <attributes>
@@
 </autorouter>
 <elements>
-<element name="U$1" library="ligocki" package="RIAA_PREAMP" value="RIAA_PREAMP" x="12" y="22" smashed="yes"/>
 <element name="A1" library="NUCLEO-F303K8" package="MODULE_NUCLEO-F303K8" value="NUCLEO-F303K8" x="175" y="43" smashed="yes">
 <attribute name="AVAILABILITY" value="Unavailable" x="175" y="43" size="1.778" layer="27" display="off"/>
@@
 <attribute name="VALUE" x="165.74381875" y="15.4816" size="1.779190625" layer="27"/>
 </element>
+<element name="U$2" library="gramofon" package="BUTTON" value="BUTTON" x="-11" y="-12" smashed="yes"/>
+<element name="U$3" library="gramofon" package="BUTTON" value="BUTTON" x="-25" y="-12" smashed="yes"/>
+<element name="U$4" library="gramofon" package="BUTTON" value="BUTTON" x="-39" y="-12" smashed="yes"/>
+<element name="U$5" library="gramofon" package="MOTOR_DRIVER" value="MOTOR_DRIVER" x="88" y="9" smashed="yes"/>
 </elements>
 <signals>
 <signal name="N$2">
-<via x="217" y="59" extent="1-16" drill="2.5" diameter="4"/>
+<via x="207" y="59" extent="1-16" drill="2.5" diameter="4"/>
 </signal>
 <signal name="N$3">
-<via x="217" y="69" extent="1-16" drill="2.5" diameter="4"/>
+<via x="207" y="69" extent="1-16" drill="2.5" diameter="4"/>
 </signal>
 <signal name="N$4">
-<via x="217" y="49" extent="1-16" drill="2.5" diameter="4"/>
+<via x="207" y="49" extent="1-16" drill="2.5" diameter="4"/>
+</signal>
+<signal name="N$1">
+<via x="209" y="74" extent="1-16" drill="2"/>
+</signal>
+<signal name="N$5">
+<via x="209" y="44" extent="1-16" drill="2"/>
+</signal>
+<signal name="N$6">
+<via x="197" y="44" extent="1-16" drill="2"/>
+</signal>
+<signal name="N$7">
+<via x="197" y="74" extent="1-16" drill="2"/>
 </signal>
 </signals>

Commit message: updated gramofon board
Parts:
- added C1, C3, C4, C5: 100n, rcl:C1206
- added C2: 100u, rcl:150CLZ-1010
- added LED1: (no value), led:1206
- added R1, R2, R3, R4: 10k, rcl:R1206
- added X1, X2, X3, X4, X5, X6, X7, X8: (no value), con-wago-500:W237-102
- moved U$4 305.9 mm to (253.0, 79.0), turned to 270 degrees
- moved U$3 288.2 mm to (253.0, 64.0), turned to 270 degrees
- moved U$2 271.0 mm to (253.0, 49.0), turned to 270 degrees
- moved U$5 69.4 mm to (155.0, 27.0), turned to 90 degrees
- moved A1 5.00 mm to (175.0, 48.0)
Connections:
- new net 3V3: A1.4.14, X6.1
- new net ADC_0: A1.4.8, X2.2
- new net ADC_1: A1.4.9, X2.1
- new net BUTT_0: C5.1, R2.1, U$4.INPUT
- new net BUTT_1: C4.1, R3.1, U$2.INPUT
- new net BUTT_2: C3.1, R4.1, U$3.INPUT
- new net GND: A1.3.4, A1.4.2, C1.2, C2.-, C3.2, C4.2, C5.2, LED1.C, U$2.PUSH_TO_ON, U$3.PUSH_TO_ON, U$4.PUSH_TO_ON, X1.2, X5.2, X6.2, X7.1, X7.2, X8.1, X8.2
- new net IO_0: A1.4.11, X4.2
- new net IO_1: A1.4.12, X4.1
- new net N$8: LED1.A, R1.1
- new net PWM_0: A1.4.6, X3.2
- new net PWM_1: A1.4.7, X3.1
- new net VCC: A1.4.1, A1.4.4, C1.1, C2.+, R1.2, R2.2, R3.2, R4.2, X1.1, X5.1
Routing:
- net GND: track 0.00 -> 355.6 mm
- net VCC: track 0.00 -> 255.7 mm
- net PWM_0: track 0.00 -> 79.9 mm
- net 3V3: track 0.00 -> 79.1 mm
- net PWM_1: track 0.00 -> 72.9 mm
- net ADC_0: track 0.00 -> 58.6 mm
- net ADC_1: track 0.00 -> 51.6 mm
- net IO_0: track 0.00 -> 35.4 mm
- net IO_1: track 0.00 -> 30.7 mm
- net BUTT_2: track 0.00 -> 12.9 mm
- net BUTT_1: track 0.00 -> 12.9 mm
- net BUTT_0: track 0.00 -> 12.9 mm
- net N$8: track 0.00 -> 5.16 mm
Other:
- board text added: "3V3"
- board text added: "5V"
- board text added: "ADC_0"
- board text added: "ADC_1"
- board text added: "GND"
- board text added: "IO_0"
- board text added: "IO_1"
- board text added: "PWM_0"
- board text added: "PWM_1"

Commit message: gramofon update
Routing:
- net GND: track 355.6 -> 357.0 mm
Changed lines of the file:
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@@
 <wire x1="222" y1="34" x2="222" y2="84" width="0.1524" layer="20"/>
 <wire x1="222" y1="84" x2="235" y2="84" width="0.1524" layer="20"/>
-<hole x="263" y="94" drill="5"/>
-<hole x="263" y="6" drill="5"/>
-<hole x="68" y="5" drill="5"/>
 <dimension x1="263" y1="94" x2="290" y2="94" x3="276.5" y3="89" textsize="1.778" layer="47"/>
 <dimension x1="263" y1="94" x2="263" y2="99" x3="258" y3="96.5" textsize="1.778" layer="47"/>
@@
 <dimension x1="222" y1="34" x2="222" y2="84" x3="240" y3="59" textsize="1.778" layer="47"/>
 <dimension x1="222" y1="84" x2="235" y2="84" x3="228.5" y3="87" textsize="1.778" layer="47"/>
-<hole x="67" y="92" drill="5"/>
 <dimension x1="67" y1="92" x2="57" y2="92" x3="62" y3="86" textsize="1.778" layer="47"/>
 <dimension x1="67" y1="92" x2="67" y2="99" x3="74" y3="95.5" textsize="1.778" layer="47"/>
@@
 <text x="143" y="14" size="1.778" layer="25" rot="R90">PWM_1</text>
 <wire x1="57" y1="86" x2="57" y2="0" width="0.8128" layer="25"/>
+<hole x="263" y="94" drill="3.2"/>
+<hole x="263" y="6" drill="3.2"/>
+<hole x="68" y="5" drill="3.2"/>
+<hole x="67" y="92" drill="3.2"/>
 </plain>
 <attributes>
@@
 <wire x1="262.6" y1="46.1" x2="262" y2="45.5" width="0.8128" layer="1"/>
 <wire x1="236.5" y1="12.5" x2="237" y2="13" width="0.8128" layer="1"/>
-<wire x1="237" y1="13" x2="261" y2="13" width="0.8128" layer="1"/>
-<wire x1="261" y1="13" x2="262" y2="14" width="0.8128" layer="1"/>
-<wire x1="262" y1="14" x2="262" y2="45.5" width="0.8128" layer="1"/>
+<wire x1="237" y1="13" x2="262" y2="13" width="0.8128" layer="1"/>
+<wire x1="262" y1="13" x2="263" y2="14" width="0.8128" layer="1"/>
+<wire x1="263" y1="44.5" x2="263" y2="14" width="0.8128" layer="1"/>
+<wire x1="263" y1="44.5" x2="262" y2="45.5" width="0.8128" layer="1"/>
 <wire x1="167.38" y1="58.16" x2="169" y2="58.16" width="0.8128" layer="1"/>
 <wire x1="169" y1="58.16" x2="173.16" y2="58.16" width="0.8128" layer="1"/>

Commit message: updated gramofon board
Parts:
- moved C4 7.21 mm to (260.0, 47.0)
- moved R3 6.71 mm to (269.0, 47.0)
- moved U$2 6.71 mm to (250.0, 43.0)
- moved C5 5.00 mm to (260.0, 86.0)
- moved C3 4.47 mm to (260.0, 66.0)
- moved R2 4.24 mm to (269.0, 86.0)
- moved U$4 4.24 mm to (250.0, 82.0)
- moved R4 3.61 mm to (269.0, 66.0)
- moved U$3 3.61 mm to (250.0, 62.0)
Routing:
- net VCC: track 255.7 -> 261.2 mm
- net GND: track 357.0 -> 360.9 mm
- net BUTT_2: track 12.9 -> 13.9 mm
- net BUTT_1: track 12.9 -> 13.9 mm
- net BUTT_0: track 12.9 -> 13.9 mm
