File: projects/gramofon/main_board.brd (EAGLE design)
At the start: 233 x 99 mm, 25 parts

Commit message: updated battery board
Parts:
- added LED2, LED3, LED4: (no value), led:CHIPLED_1206
- added R5, R6, R7: 10k, rcl:R1206
- moved X11 107.7 mm to (79.0, 8.00), turned to 180 degrees
- moved X10 83.9 mm to (66.0, 8.00), turned to 180 degrees
- moved X7 64.0 mm to (53.0, 8.00)
- moved X8 64.0 mm to (43.0, 8.00)
- moved A1 57.0 mm to (118.0, 48.0)
- moved C1 57.0 mm to (139.0, 17.0)
- moved C2 57.0 mm to (139.0, 29.0)
- moved C3 57.0 mm to (203.0, 66.0)
- moved C4 57.0 mm to (203.0, 47.0)
- moved C5 57.0 mm to (203.0, 86.0)
- moved LED1 57.0 mm to (143.0, 21.0)
- moved R1 57.0 mm to (135.0, 21.0)
- moved R2 57.0 mm to (212.0, 86.0)
- moved R3 57.0 mm to (212.0, 47.0)
- moved R4 57.0 mm to (212.0, 66.0)
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Connections:
- new net N$11: LED4.A, R7.2
- new net N$12: LED3.A, R6.2
- new net N$13: LED2.A, R5.2
- new net N$2: A1.3.9, LED2.C
- new net N$3: A1.3.8, LED3.C
- new net N$4: A1.3.7, LED4.C
- net IO_2: now also A1.3.14; no longer A1.3.15
- net IO_3: now also A1.3.15; no longer A1.3.14
- net VCC: now also R5.1, R6.1, R7.1
Routing:
- net PWM_2: track 0.00 -> 102.2 mm
- net PWM_3: track 0.00 -> 94.8 mm
- net IO_2: track 0.00 -> 52.5 mm
- net IO_3: track 0.00 -> 45.9 mm
- net VCC: track 261.2 -> 305.3 mm, vias 0 -> 2
- net PWM_0: track 79.9 -> 69.9 mm
- net PWM_1: track 72.9 -> 63.5 mm
- net ADC_0: track 58.6 -> 53.6 mm
- net ADC_1: track 51.6 -> 46.6 mm
- net N$13: track 0.00 -> 4.83 mm, vias 0 -> 1
- net N$12: track 0.00 -> 4.83 mm, vias 0 -> 1
- net N$11: track 0.00 -> 4.83 mm, vias 0 -> 1
- net N$4: track 0.00 -> 4.82 mm
- net N$2: track 0.00 -> 4.82 mm
- net N$3: track 0.00 -> 4.63 mm
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Other:
- outline, holes or cut-outs redrawn
- board text added: "IO_2"
- board text added: "IO_3"
- board text added: "PWM_2"
- board text added: "PWM_3"
